File: hardware/KiCad/sdbox.sch (KiCad schematic (older format))
At the start: 21 parts, among them J1 DB25_Male_MountingHoles, J2 Barrel_Jack, J3 Conn_01x01, J4 Conn_01x01, J5 Conn_01x01, J6 Conn_01x01, Q1 BC847BW, Q2 BC847BW, U1 Arduino_Nano_V3, U2 Micro_SD_Card_Module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

Commit message: fixed symbol and footprint libs now included as project libs
Parts:
- R5: footprint Capacitor_SMD:C_1206_3216Metric_Pad1.42x1.75mm_HandSolder -> Resistor_SMD:R_1206_3216Metric_Pad1.42x1.75mm_HandSolder
- U1: footprint Arduino:Arduino_Nano_V3_Schield -> sdbox:Arduino_Nano_V3_Schield; symbol MCU_Microchip_AVR:Arduino_Nano_V3 -> sdbox:Arduino_Nano_V3
- U2: symbol Connector:Micro_SD_Card_Module -> sdbox:Micro_SD_Card_Module
- U3: footprint Relay_SMD:SOIC254P978X443-6N -> sdbox:SOIC254P978X443-6N; symbol Relay_SolidState:PVG612S -> sdbox:PVG612S
Other:
- note added: "Optional for powering on/off \nwith the Amiga’s on/off"
- note removed: "Optional for power down when \nAmiga is shutdown"
Changed lines of the file:
@@
 EESchema Schematic File Version 4
-LIBS:sdbox-cache
-EELAYER 29 0
+EELAYER 30 0
 EELAYER END
 $Descr A4 11693 8268
@@
 GND
 $Comp
-L Connector:Micro_SD_Card_Module U2
+L sdbox:Micro_SD_Card_Module U2
 U 1 1 5EB40C39
 P 7050 4900
@@
 SCK
 $Comp
-L MCU_Microchip_AVR:Arduino_Nano_V3 U1
+L sdbox:Arduino_Nano_V3 U1
 U 1 1 5EB5B4AA
 P 5450 4100
 F 0 "U1" H 5450 4250 50  0000 C CNN
 F 1 "Arduino_Nano_V3" H 5950 3050 50  0000 C CNN
-F 2 "Arduino:Arduino_Nano_V3_Schield" H 5450 4100 50  0001 C CNN
+F 2 "sdbox:Arduino_Nano_V3_Schield" H 5450 4100 50  0001 C CNN
 F 3 "" H 5450 4100 50  0001 C CNN
 	1    5450 4100
@@
 MOSI
 $Comp
-L Relay_SolidState:PVG612S U3
+L sdbox:PVG612S U3
 U 1 1 5EB77D01
 P 6050 2650
 F 0 "U3" H 6050 2450 50  0000 C CNN
 F 1 "PVG612S" H 6050 2950 50  0000 C CNN
-F 2 "Relay_SMD:SOIC254P978X443-6N" H 6120 3225 50  0001 C CNN
-F 3 "" H 6120 3225 50  0001 C CNN
+F 2 "sdbox:SOIC254P978X443-6N" H 6120 3225 50  0001 C CNN
+F 3 "https://www.infineon.com/dgdl/Infineon-PVG612-DataSheet-v01_00-EN.pdf?fileId=5546d462533600a401535683c1892937" H 6120 3225 50  0001 C CNN
 	1    6050 2650
 	1    0    0    -1
@@
 	6150 3650 6450 3650
 Text Notes 5200 2250 0    50   ~ 0
-Optional for power down when \nAmiga is shutdown
+Optional for powering on/off \nwith the Amiga’s on/off
 NoConn ~ 4800 3950
 NoConn ~ 4800 4450
@@
 Wire Notes Line
 	6600 2300 8100 2300
-Wire Notes Line
-	6600 3000 8100 3000
 Text Notes 5390 5030 1    50   ~ 0
 VCC\n
@@
 Amiga5V
 Wire Notes Line
-	6550 2050 6550 2950
-Wire Notes Line
 	5100 2050 5100 2950
 $Comp
@@
 F 0 "R5" V 5546 2500 50  0000 C CNN
 F 1 "R_Small" V 5545 2500 50  0001 C CNN
-F 2 "Capacitor_SMD:C_1206_3216Metric_Pad1.42x1.75mm_HandSolder" H 5650 2500 50  0001 C CNN
+F 2 "Resistor_SMD:R_1206_3216Metric_Pad1.42x1.75mm_HandSolder" H 5650 2500 50  0001 C CNN
 F 3 "~" H 5650 2500 50  0001 C CNN
 	1    5650 2500
@@
 NoConn ~ 5550 5550
 NoConn ~ 5150 5550
-Wire Notes Line
-	6550 2950 5100 2950
 Wire Notes Line
 	6550 2050 5100 2050
@@
 Wire Notes Line
 	7500 3050 7500 4450
+Wire Notes Line
+	6550 2950 5100 2950
+Wire Notes Line
+	6550 2050 6550 2950
+Wire Notes Line
+	6600 3000 6850 3000
+Wire Notes Line
+	6850 3000 6850 3250
+Wire Notes Line
+	6850 3250 6200 3250
+Wire Notes Line
+	6200 3250 6200 3450
+Wire Notes Line
+	6200 3450 7450 3450
+Wire Notes Line
+	7450 3450 7450 3000
+Wire Notes Line
+	7450 3000 8100 3000
 $EndSCHEMATC
